Commit message: 3 wheeled robot

File: description/gazebo_control.xacro (robot description, xacro)
@@ -4,8 +4,10 @@
         <plugin name="wheel_drive_controller" filename="libgazebo_ros_diff_drive.so">
             <!-- wheels -->
-            <num_wheel_pairs>2</num_wheel_pairs>
+            <num_wheel_pairs>3</num_wheel_pairs>
             <right_joint>front_right_wheel_joint</right_joint>
+            <right_joint>middle_right_wheel_joint</right_joint>
             <right_joint>back_right_wheel_joint</right_joint>
             <left_joint>front_left_wheel_joint</left_joint>
+            <left_joint>middle_left_wheel_joint</left_joint>
             <left_joint>back_left_wheel_joint</left_joint>
             <!-- kinematics -->

File: description/robot_core.xacro (robot description, xacro)
@@ -53,9 +53,113 @@
         <material>Gazebo/Red</material>
     </gazebo>
+<!-- front_left wheel link -->
+    <joint name="front_left_wheel_joint" type="continuous">
+        <parent link="chassis"/>
+        <child link="front_left_wheel"/>
+        <origin xyz="0.285 0.175 -0.08" rpy="-${pi/2} 0 0"/>
+        <axis xyz="0 0 1"/>
+    </joint>
+    <link name="front_left_wheel">
+        <visual>
+            <geometry>
+                <cylinder radius="0.05" length="0.04"/>
+            </geometry>
+            <material name="black"/>
+        </visual>
+        <collision>
+            <geometry>
+                <cylinder radius="0.05" length="0.04"/>
+            </geometry>
+        </collision>
+        <xacro:inertial_cylinder mass="0.1" length="0.04" radius="0.05">
+            <origin xyz="0 0 0" rpy="0 0 0"/>
+        </xacro:inertial_cylinder>
+    </link>
+    <gazebo reference="front_left_wheel">
+        <material>Gazebo/Blue</material>
+    </gazebo>
+<!-- front Right wheel link -->
+    <joint name="front_right_wheel_joint" type="continuous">
+        <parent link="chassis"/>
+        <child link="front_right_wheel"/>
+        <origin xyz="0.285 -0.175 -0.08" rpy="${pi/2} 0 0"/>
+        <axis xyz="0 0 -1"/>
+    </joint>
+    <link name="front_right_wheel">
+        <visual>
+            <geometry>
+                <cylinder radius="0.05" length="0.04"/>
+            </geometry>
+            <material name="black"/>
+        </visual>
+        <collision>
+            <geometry>
+                <cylinder radius="0.05" length="0.04"/>
+            </geometry>
+        </collision>
+        <xacro:inertial_cylinder mass="0.1" length="0.04" radius="0.05">
+            <origin xyz="0 0 0" rpy="0 0 0"/>
+        </xacro:inertial_cylinder>
+    </link>
+    <gazebo reference="front_right_wheel">
+        <material>Gazebo/Blue</material>
+    </gazebo>
+    <!-- middle_left wheel link -->
+    <joint name="middle_left_wheel_joint" type="continuous">
+        <parent link="chassis"/>
+        <child link="middle_left_wheel"/>
+        <origin xyz="0.150 0.175 -0.08" rpy="-${pi/2} 0 0"/>
+        <axis xyz="0 0 1"/>
+    </joint>
+    <link name="middle_left_wheel">
+        <visual>
+            <geometry>
+                <cylinder radius="0.05" length="0.04"/>
+            </geometry>
+            <material name="black"/>
+        </visual>
+        <collision>
+            <geometry>
+                <cylinder radius="0.05" length="0.04"/>
+            </geometry>
+        </collision>
+        <xacro:inertial_cylinder mass="0.1" length="0.04" radius="0.05">
+            <origin xyz="0 0 0" rpy="0 0 0"/>
+        </xacro:inertial_cylinder>
+    </link>
+    <gazebo reference="middle_left_wheel">
+        <material>Gazebo/Blue</material>
+    </gazebo>
+<!-- middle Right wheel link -->
+    <joint name="middle_right_wheel_joint" type="continuous">
+        <parent link="chassis"/>
+        <child link="middle_right_wheel"/>
+        <origin xyz="0.150 -0.175 -0.08" rpy="${pi/2} 0 0"/>
+        <axis xyz="0 0 -1"/>
+    </joint>
+    <link name="middle_right_wheel">
+        <visual>
+            <geometry>
+                <cylinder radius="0.05" length="0.04"/>
+            </geometry>
+            <material name="black"/>
+        </visual>
+        <collision>
+            <geometry>
+                <cylinder radius="0.05" length="0.04"/>
+            </geometry>
+        </collision>
+        <xacro:inertial_cylinder mass="0.1" length="0.04" radius="0.05">
+            <origin xyz="0 0 0" rpy="0 0 0"/>
+        </xacro:inertial_cylinder>
+    </link>
+    <gazebo reference="middle_right_wheel">
+        <material>Gazebo/Blue</material>
+    </gazebo>
 <!-- back left wheel link -->
     <joint name="back_left_wheel_joint" type="continuous">
-        <parent link="base_link"/>
+        <parent link="chassis"/>
         <child link="back_left_wheel"/>
-        <origin xyz="-0.068 0.175 -0.08" rpy="-${pi/2} 0 0"/>
+        <origin xyz="0.015 0.175 -0.08" rpy="-${pi/2} 0 0"/>
         <axis xyz="0 0 1"/>
     </joint>
@@ -81,7 +185,7 @@
 <!-- back Right wheel link -->
     <joint name="back_right_wheel_joint" type="continuous">
-        <parent link="base_link"/>
+        <parent link="chassis"/>
         <child link="back_right_wheel"/>
-        <origin xyz="-0.068 -0.175 -0.08" rpy="${pi/2} 0 0"/>
+        <origin xyz="0.015 -0.175 -0.08" rpy="${pi/2} 0 0"/>
         <axis xyz="0 0 -1"/>
     </joint>
@@ -105,55 +209,3 @@
         <material>Gazebo/Blue</material>
     </gazebo>
-<!-- front_left wheel link -->
-    <joint name="front_left_wheel_joint" type="continuous">
-        <parent link="base_link"/>
-        <child link="front_left_wheel"/>
-        <origin xyz="0.165 0.175 -0.08" rpy="-${pi/2} 0 0"/>
-        <axis xyz="0 0 1"/>
-    </joint>
-    <link name="front_left_wheel">
-        <visual>
-            <geometry>
-                <cylinder radius="0.05" length="0.04"/>
-            </geometry>
-            <material name="black"/>
-        </visual>
-        <collision>
-            <geometry>
-                <cylinder radius="0.05" length="0.04"/>
-            </geometry>
-        </collision>
-        <xacro:inertial_cylinder mass="0.1" length="0.04" radius="0.05">
-            <origin xyz="0 0 0" rpy="0 0 0"/>
-        </xacro:inertial_cylinder>
-    </link>
-    <gazebo reference="front_left_wheel">
-        <material>Gazebo/Blue</material>
-    </gazebo>
-<!-- front Right wheel link -->
-    <joint name="front_right_wheel_joint" type="continuous">
-        <parent link="base_link"/>
-        <child link="front_right_wheel"/>
-        <origin xyz="0.165 -0.175 -0.08" rpy="${pi/2} 0 0"/>
-        <axis xyz="0 0 -1"/>
-    </joint>
-    <link name="front_right_wheel">
-        <visual>
-            <geometry>
-                <cylinder radius="0.05" length="0.04"/>
-            </geometry>
-            <material name="black"/>
-        </visual>
-        <collision>
-            <geometry>
-                <cylinder radius="0.05" length="0.04"/>
-            </geometry>
-        </collision>
-        <xacro:inertial_cylinder mass="0.1" length="0.04" radius="0.05">
-            <origin xyz="0 0 0" rpy="0 0 0"/>
-        </xacro:inertial_cylinder>
-    </link>
-    <gazebo reference="front_right_wheel">
-        <material>Gazebo/Blue</material>
-    </gazebo>
 </robot>
